File: DroneV1/Sensors.sch (KiCad schematic (older format))
At the start: 9 parts

Commit message: Added indicator LEDs
Parts:
- C10, C11, C12, C13, C14, C15: renamed from C?; footprint (none) -> Capacitor_SMD:C_0603_1608Metric
- R20: renamed from R?; footprint (none) -> Resistor_SMD:R_0603_1608Metric
- gave numbers to parts that had none: 2
Changed lines of the file:
@@
 $EndDescr
 $Comp
-L Sensor_Pressure:BMP280 U?
+L Sensor_Pressure:BMP280 U3
 U 1 1 5E00419A
 P 2600 2950
-F 0 "U?" H 2830 3046 50  0000 L CNN
+F 0 "U3" H 2830 3046 50  0000 L CNN
 F 1 "BMP280" H 2830 2955 50  0000 L CNN
 F 2 "Package_LGA:Bosch_LGA-8_2x2.5mm_P0.65mm_ClockwisePinNumbering" H 2600 2250 50  0001 C CNN
@@
 $EndComp
 $Comp
-L Sensor_Motion:MPU-6050 U?
+L Sensor_Motion:MPU-6050 U4
 U 1 1 5E004571
 P 6050 2850
-F 0 "U?" H 5600 2050 50  0000 C CNN
+F 0 "U4" H 5600 2050 50  0000 C CNN
 F 1 "MPU-6050" H 5750 1950 50  0000 C CNN
 F 2 "Sensor_Motion:InvenSense_QFN-24_4x4mm_P0.5mm" H 6050 2050 50  0001 C CNN
@@
 $EndComp
 $Comp
-L Device:C C?
+L Device:C C11
 U 1 1 5E0046B5
 P 2850 2400
-F 0 "C?" V 2598 2400 50  0000 C CNN
+F 0 "C11" V 2598 2400 50  0000 C CNN
 F 1 "100nF" V 2689 2400 50  0000 C CNN
-F 2 "" H 2888 2250 50  0001 C CNN
+F 2 "Capacitor_SMD:C_0603_1608Metric" H 2888 2250 50  0001 C CNN
 F 3 "~" H 2850 2400 50  0001 C CNN
 	1    2850 2400
@@
 $EndComp
 $Comp
-L Device:C C?
+L Device:C C10
 U 1 1 5E004AFE
 P 2450 2400
-F 0 "C?" V 2198 2400 50  0000 C CNN
+F 0 "C10" V 2198 2400 50  0000 C CNN
 F 1 "100nF" V 2289 2400 50  0000 C CNN
-F 2 "" H 2488 2250 50  0001 C CNN
+F 2 "Capacitor_SMD:C_0603_1608Metric" H 2488 2250 50  0001 C CNN
 F 3 "~" H 2450 2400 50  0001 C CNN
 	1    2450 2400
@@
 Connection ~ 2600 2400
 $Comp
-L power:VBUS #PWR?
+L power:VBUS #PWR049
 U 1 1 5E005190
 P 2600 2400
-F 0 "#PWR?" H 2600 2250 50  0001 C CNN
+F 0 "#PWR049" H 2600 2250 50  0001 C CNN
 F 1 "VBUS" H 2650 2650 50  0000 C CNN
 F 2 "" H 2600 2400 50  0001 C CNN
@@
 $EndComp
 $Comp
-L power:GND #PWR?
+L power:GND #PWR051
 U 1 1 5E0052BC
 P 3000 2400
-F 0 "#PWR?" H 3000 2150 50  0001 C CNN
+F 0 "#PWR051" H 3000 2150 50  0001 C CNN
 F 1 "GND" H 3005 2227 50  0000 C CNN
 F 2 "" H 3000 2400 50  0001 C CNN
@@
 $EndComp
 $Comp
-L power:GND #PWR?
+L power:GND #PWR048
 U 1 1 5E0053D0
 P 2300 2400
-F 0 "#PWR?" H 2300 2150 50  0001 C CNN
+F 0 "#PWR048" H 2300 2150 50  0001 C CNN
 F 1 "GND" H 2305 2227 50  0000 C CNN
 F 2 "" H 2300 2400 50  0001 C CNN
@@
 SDA
 $Comp
-L power:GND #PWR?
+L power:GND #PWR050
 U 1 1 5E005644
 P 2600 3250
-F 0 "#PWR?" H 2600 3000 50  0001 C CNN
+F 0 "#PWR050" H 2600 3000 50  0001 C CNN
 F 1 "GND" H 2605 3077 50  0000 C CNN
 F 2 "" H 2600 3250 50  0001 C CNN
@@
 Connection ~ 2600 3250
 $Comp
-L power:GND #PWR?
+L power:GND #PWR046
 U 1 1 5E00585E
 P 2200 2950
-F 0 "#PWR?" H 2200 2700 50  0001 C CNN
+F 0 "#PWR046" H 2200 2700 50  0001 C CNN
 F 1 "GND" V 2205 2822 50  0000 R CNN
 F 2 "" H 2200 2950 50  0001 C CNN
@@
 $EndComp
 $Comp
-L power:+3.3V #PWR?
+L power:+3.3V #PWR047
 U 1 1 5E005D1C
 P 2200 3050
-F 0 "#PWR?" H 2200 2900 50  0001 C CNN
+F 0 "#PWR047" H 2200 2900 50  0001 C CNN
 F 1 "+3.3V" V 2215 3178 50  0000 L CNN
 F 2 "" H 2200 3050 50  0001 C CNN
@@
 SCL
 $Comp
-L power:GND #PWR?
+L power:GND #PWR052
 U 1 1 5E0064B7
 P 5350 3150
-F 0 "#PWR?" H 5350 2900 50  0001 C CNN
+F 0 "#PWR052" H 5350 2900 50  0001 C CNN
 F 1 "GND" H 5355 2977 50  0000 C CNN
 F 2 "" H 5350 3150 50  0001 C CNN
@@
 Connection ~ 5350 3150
 $Comp
-L Device:R R?
+L Device:R R20
 U 1 1 5E00675E
 P 5350 2900
-F 0 "R?" H 5150 2950 50  0000 L CNN
+F 0 "R20" H 5150 2950 50  0000 L CNN
 F 1 "4.7k" H 5150 2850 50  0000 L CNN
-F 2 "" V 5280 2900 50  0001 C CNN
+F 2 "Resistor_SMD:R_0603_1608Metric" V 5280 2900 50  0001 C CNN
 F 3 "~" H 5350 2900 50  0001 C CNN
 	1    5350 2900
@@
 Connection ~ 5350 3050
 $Comp
-L Device:C C?
+L Device:C C12
 U 1 1 5E0083C3
 P 5800 2000
-F 0 "C?" V 5548 2000 50  0000 C CNN
+F 0 "C12" V 5548 2000 50  0000 C CNN
 F 1 "10nF" V 5639 2000 50  0000 C CNN
-F 2 "" H 5838 1850 50  0001 C CNN
+F 2 "Capacitor_SMD:C_0603_1608Metric" H 5838 1850 50  0001 C CNN
 F 3 "~" H 5800 2000 50  0001 C CNN
 	1    5800 2000
@@
 $EndComp
 $Comp
-L Device:C C?
+L Device:C C13
 U 1 1 5E00891E
 P 6300 2000
-F 0 "C?" V 6048 2000 50  0000 C CNN
+F 0 "C13" V 6048 2000 50  0000 C CNN
 F 1 "100nF" V 6139 2000 50  0000 C CNN
-F 2 "" H 6338 1850 50  0001 C CNN
+F 2 "Capacitor_SMD:C_0603_1608Metric" H 6338 1850 50  0001 C CNN
 F 3 "~" H 6300 2000 50  0001 C CNN
 	1    6300 2000
@@
 $EndComp
 $Comp
-L power:GND #PWR?
+L power:GND #PWR053
 U 1 1 5E008DCC
 P 5650 2000
-F 0 "#PWR?" H 5650 1750 50  0001 C CNN
+F 0 "#PWR053" H 5650 1750 50  0001 C CNN
 F 1 "GND" H 5655 1827 50  0000 C CNN
 F 2 "" H 5650 2000 50  0001 C CNN
@@
 $EndComp
 $Comp
-L power:GND #PWR?
+L power:GND #PWR056
 U 1 1 5E008F62
 P 6450 2000
-F 0 "#PWR?" H 6450 1750 50  0001 C CNN
+F 0 "#PWR056" H 6450 1750 50  0001 C CNN
 F 1 "GND" H 6455 1827 50  0000 C CNN
 F 2 "" H 6450 2000 50  0001 C CNN
@@
 $EndComp
 $Comp
-L power:+3.3V #PWR?
+L power:+3.3V #PWR054
 U 1 1 5E00912F
 P 6050 1800
-F 0 "#PWR?" H 6050 1650 50  0001 C CNN
+F 0 "#PWR054" H 6050 1650 50  0001 C CNN
 F 1 "+3.3V" H 6065 1973 50  0000 C CNN
 F 2 "" H 6050 1800 50  0001 C CNN
@@
 	6050 2000 5950 2000
 $Comp
-L power:GND #PWR?
+L power:GND #PWR055
 U 1 1 5E009B6B
 P 6050 3550
-F 0 "#PWR?" H 6050 3300 50  0001 C CNN
+F 0 "#PWR055" H 6050 3300 50  0001 C CNN
 F 1 "GND" H 6055 3377 50  0000 C CNN
 F 2 "" H 6050 3550 50  0001 C CNN
@@
 $EndComp
 $Comp
-L Device:C C?
+L Device:C C14
 U 1 1 5E00A088
 P 6750 3300
-F 0 "C?" H 6635 3254 50  0000 R CNN
+F 0 "C14" H 6635 3254 50  0000 R CNN
 F 1 "100nF" H 6635 3345 50  0000 R CNN
-F 2 "" H 6788 3150 50  0001 C CNN
+F 2 "Capacitor_SMD:C_0603_1608Metric" H 6788 3150 50  0001 C CNN
 F 3 "~" H 6750 3300 50  0001 C CNN
 	1    6750 3300
@@
 $EndComp
 $Comp
-L power:GND #PWR?
+L power:GND #PWR057
 U 1 1 5E00A3D7
 P 6750 3450
-F 0 "#PWR?" H 6750 3200 50  0001 C CNN
+F 0 "#PWR057" H 6750 3200 50  0001 C CNN
 F 1 "GND" H 6755 3277 50  0000 C CNN
 F 2 "" H 6750 3450 50  0001 C CNN
@@
 $EndComp
 $Comp
-L Device:C C?
+L Device:C C15
 U 1 1 5E00B55B
 P 7250 3300
-F 0 "C?" H 7135 3254 50  0000 R CNN
+F 0 "C15" H 7135 3254 50  0000 R CNN
 F 1 "2.2nF" H 7135 3345 50  0000 R CNN
-F 2 "" H 7288 3150 50  0001 C CNN
+F 2 "Capacitor_SMD:C_0603_1608Metric" H 7288 3150 50  0001 C CNN
 F 3 "~" H 7250 3300 50  0001 C CNN
 	1    7250 3300
@@
 $EndComp
 $Comp
-L power:GND #PWR?
+L power:GND #PWR058
 U 1 1 5E00B9A1
 P 7250 3450
-F 0 "#PWR?" H 7250 3200 50  0001 C CNN
+F 0 "#PWR058" H 7250 3200 50  0001 C CNN
 F 1 "GND" H 7255 3277 50  0000 C CNN
 F 2 "" H 7250 3450 50  0001 C CNN
