File: DroneV1/motorsAndController.sch (KiCad schematic (older format))
At the start: 18 parts, among them IC1 74HC14D,652, M1 Motor_DC, M2 Motor_DC, M3 Motor_DC, M4 Motor_DC, Q1 DMHC3025LSD-13, Q2 DMHC3025LSD-13, Q3 DMHC3025LSD-13, Q4 DMHC3025LSD-13

Commit message: Added indicator LEDs
Parts:
- C1: footprint (none) -> Capacitor_SMD:C_0603_1608Metric
- IC1: footprint (none) -> Package_DIP:DIP-14_W7.62mm
- M1, M2, M3, M4: footprint (none) -> Connector_PinHeader_2.54mm:PinHeader_1x02_P2.54mm_Vertical
Changed lines of the file:
@@
 F 0 "M1" H 1558 2196 50  0000 L CNN
 F 1 "Motor_DC" H 1558 2105 50  0000 L CNN
-F 2 "" H 1400 2110 50  0001 C CNN
+F 2 "Connector_PinHeader_2.54mm:PinHeader_1x02_P2.54mm_Vertical" H 1400 2110 50  0001 C CNN
 F 3 "~" H 1400 2110 50  0001 C CNN
 	1    1400 2200
@@
 F 0 "M2" H 1558 4046 50  0000 L CNN
 F 1 "Motor_DC" H 1558 3955 50  0000 L CNN
-F 2 "" H 1400 3960 50  0001 C CNN
+F 2 "Connector_PinHeader_2.54mm:PinHeader_1x02_P2.54mm_Vertical" H 1400 3960 50  0001 C CNN
 F 3 "~" H 1400 3960 50  0001 C CNN
 	1    1400 4050
@@
 F 0 "M3" H 4658 2196 50  0000 L CNN
 F 1 "Motor_DC" H 4658 2105 50  0000 L CNN
-F 2 "" H 4500 2110 50  0001 C CNN
+F 2 "Connector_PinHeader_2.54mm:PinHeader_1x02_P2.54mm_Vertical" H 4500 2110 50  0001 C CNN
 F 3 "~" H 4500 2110 50  0001 C CNN
 	1    4500 2200
@@
 F 0 "M4" H 4658 4046 50  0000 L CNN
 F 1 "Motor_DC" H 4658 3955 50  0000 L CNN
-F 2 "" H 4500 3960 50  0001 C CNN
+F 2 "Connector_PinHeader_2.54mm:PinHeader_1x02_P2.54mm_Vertical" H 4500 3960 50  0001 C CNN
 F 3 "~" H 4500 3960 50  0001 C CNN
 	1    4500 4050
@@
 F 0 "C1" H 8365 2046 50  0000 L CNN
 F 1 "C" H 8365 1955 50  0000 L CNN
-F 2 "" H 8288 1850 50  0001 C CNN
+F 2 "Capacitor_SMD:C_0603_1608Metric" H 8288 1850 50  0001 C CNN
 F 3 "~" H 8250 2000 50  0001 C CNN
 	1    8250 2000
@@
 F 0 "IC1" H 8750 3465 50  0000 C CNN
 F 1 "74HC14D,652" H 8750 3374 50  0000 C CNN
-F 2 "" H 9100 3300 50  0001 L CNN
+F 2 "Package_DIP:DIP-14_W7.62mm" H 9100 3300 50  0001 L CNN
 F 3 "https://assets.nexperia.com/documents/data-sheet/74HC_HCT14.pdf" H 9100 3200 50  0001 L CNN
 F 4 "74HC14D,652, Hex Schmitt Trigger Inverter, HC, 5.2mA 2 to 6V 14-Pin SOIC" H 9100 3100 50  0001 L CNN "Description"
